Commit message: Added FD scanner simulation

File: rrt_nbv_exploration_plugins/urdf/husky.urdf.xacro (robot description, xacro)
@@ -28,5 +28,5 @@
 	<xacro:arg name="laser_rpy"
 		default="$(optenv HUSKY_LMS1XX_RPY 0.0 0.0 0.0)" />
-	<xacro:arg name="kinect_enabled" default="true" />
+	<xacro:arg name="kinect_enabled" default="false" />
 	<xacro:arg name="kinect_xyz"
 		default="$(optenv HUSKY_KINECT_XYZ 0 0 0)" />
@@ -37,4 +37,9 @@
 	<xacro:property name="husky_rear_bumper_extend"
 		value="$(optenv HUSKY_REAR_BUMPER_EXTEND 0)" />
+	<xacro:arg name="fd_scanner_enabled" default="false" />
+	<xacro:arg name="fd_scanner_xyz"
+		default="$(optenv HUSKY_FD_SCANNER_XYZ -0.3 0 0)" />
+	<xacro:arg name="fd_scanner_rpy"
+		default="$(optenv HUSKY_FD_SCANNER_RPY 0 0 0)" />
 	<xacro:arg name="robot_namespace" default="/" />
 	<xacro:arg name="urdf_extras" default="empty.urdf" />
@@ -50,4 +55,6 @@
 	<xacro:include
 		filename="$(find rrt_nbv_exploration_plugins)/urdf/sensor_arch.urdf.xacro" />
+	<xacro:include
+		filename="$(find fd_scanner)/urdf/fd_scanner.urdf.xacro" />
 	<xacro:property name="M_PI" value="3.14159" />
 	<!-- Base Size -->
@@ -157,5 +164,5 @@
 		<joint name="camera_swivel" type="revolute">
 			<axis xyz="0 0 1" />
-			<limit upper="1.3" lower="-1.3" velocity="0.87" effort="1"/>
+			<limit upper="1.3" lower="-1.3" velocity="0.87" effort="1" />
 			<origin xyz="$(arg kinect_xyz)" rpy="$(arg kinect_rpy)" />
 			<parent link="sensor_arch_mount_link" />
@@ -174,4 +181,15 @@
 			robot_namespace="$(arg robot_namespace)" />
 	</xacro:if>
+	<xacro:if value="$(arg fd_scanner_enabled)">
+		<fd_scanner prefix="fd_scanner"
+			robot_namespace="$(arg robot_namespace)"
+			simulated_velodyne="true" />
+		<joint name="fd_scanner_joint" type="fixed">
+			<origin xyz="$(arg fd_scanner_xyz)"
+				rpy="$(arg fd_scanner_rpy)" />
+			<parent link="top_plate_link" />
+			<child link="fd_scanner_link" />
+		</joint>
+	</xacro:if>
 	<gazebo>
 		<plugin name="gazebo_ros_control"

Commit message: Changed to RealSense simulated camera

File: rrt_nbv_exploration_plugins/urdf/husky.urdf.xacro (robot description, xacro)
@@ -28,9 +28,9 @@
 	<xacro:arg name="laser_rpy"
 		default="$(optenv HUSKY_LMS1XX_RPY 0.0 0.0 0.0)" />
-	<xacro:arg name="kinect_enabled" default="false" />
-	<xacro:arg name="kinect_xyz"
-		default="$(optenv HUSKY_KINECT_XYZ 0 0 0)" />
-	<xacro:arg name="kinect_rpy"
-		default="$(optenv HUSKY_KINECT_RPY 0 0.18 3.14)" />
+	<xacro:arg name="realsense_enabled" default="false" />
+	<xacro:arg name="realsense_xyz"
+		default="$(optenv HUSKY_REALSENSE_XYZ 0 0 0)" />
+	<xacro:arg name="realsense_rpy"
+		default="$(optenv HUSKY_REALSENSE_RPY 0 0.18 3.14)" />
 	<xacro:property name="husky_front_bumper_extend"
 		value="$(optenv HUSKY_FRONT_BUMPER_EXTEND 0)" />
@@ -50,5 +50,5 @@
 		filename="$(find husky_description)/urdf/wheel.urdf.xacro" />
 	<xacro:include
-		filename="$(find rrt_nbv_exploration_plugins)/urdf/kinect_camera.urdf.xacro" />
+		filename="$(find rrt_nbv_exploration_plugins)/urdf/intel_realsense.urdf.xacro" />
 	<xacro:include
 		filename="$(find husky_description)/urdf/accessories/sick_lms1xx_mount.urdf.xacro" />
@@ -158,14 +158,31 @@
 		</joint>
 	</xacro:if>
-	<xacro:if value="$(arg kinect_enabled)">
+	<xacro:if value="$(arg realsense_enabled)">
 		<xacro:sensor_arch prefix="" parent="top_plate_link">
 			<origin xyz="-0.35 0 0.51" rpy="0 0 -3.14" />
 		</xacro:sensor_arch>
+		<link name="realsense_mountpoint">
+			<visual>
+				<geometry>
+					<box size="0.01 0.01 0.01" />
+				</geometry>
+			</visual>
+			<collision>
+				<geometry>
+					<box size="0.01 0.01 0.01" />
+				</geometry>
+			</collision>
+			<inertial>
+				<mass value="0.01" />
+				<inertia ixx="1e-3" ixy="1e-3" ixz="1e-3" iyy="1e-3"
+					iyz="1e-3" izz="1e-3" />
+			</inertial>
+		</link>
 		<joint name="camera_swivel" type="revolute">
 			<axis xyz="0 0 1" />
 			<limit upper="1.3" lower="-1.3" velocity="0.87" effort="1" />
-			<origin xyz="$(arg kinect_xyz)" rpy="$(arg kinect_rpy)" />
+			<origin xyz="$(arg realsense_xyz)" rpy="$(arg realsense_rpy)" />
 			<parent link="sensor_arch_mount_link" />
-			<child link="camera_link" />
+			<child link="realsense_mountpoint" />
 		</joint>
 		<transmission name="camera_swivel_trans">
@@ -178,6 +195,6 @@
 			</joint>
 		</transmission>
-		<xacro:kinect_camera prefix="camera"
-			robot_namespace="$(arg robot_namespace)" />
+		<xacro:intel_realsense_mount
+			prefix="camera" topic="camera" parent_link="realsense_mountpoint" />
 	</xacro:if>
 	<xacro:if value="$(arg fd_scanner_enabled)">
