Commit message: Replaced FD scanner with normal Velodyne, added warning for vertical FoV top and bottom

File: rrg_nbv_exploration_plugins/urdf/husky.urdf.xacro (robot description, xacro)
@@ -37,10 +37,5 @@
 	<xacro:property name="husky_rear_bumper_extend"
 		value="$(optenv HUSKY_REAR_BUMPER_EXTEND 0)" />
-	<xacro:arg name="fd_scanner_enabled" default="false" />
-	<xacro:arg name="fd_scanner_angled" default="false" />
-	<xacro:arg name="fd_scanner_xyz"
-		default="$(optenv HUSKY_FD_SCANNER_XYZ -0.3 0 0)" />
-	<xacro:arg name="fd_scanner_rpy"
-		default="$(optenv HUSKY_FD_SCANNER_RPY 0 0 0)" />
+	<xacro:arg name="velodyne_enabled" default="false" />
 	<xacro:arg name="robot_namespace" default="/" />
 	<!-- Included URDF/XACRO Files -->
@@ -56,6 +51,9 @@
 		filename="$(find rrg_nbv_exploration_plugins)/urdf/sensor_arch.urdf.xacro" />
 	<xacro:include
-		filename="$(find fd_scanner)/urdf/fd_scanner.urdf.xacro" />
+		filename="$(find velodyne_description)/urdf/VLP-16.urdf.xacro" />
 	<xacro:property name="M_PI" value="3.14159" />
+	<material name="black000">
+		<color rgba="0 0 0 1" />
+	</material>
 	<!-- Base Size -->
 	<xacro:property name="base_x_size" value="0.98740000" />
@@ -198,15 +196,32 @@
 			prefix="camera" topic="camera" parent_link="realsense_mountpoint" />
 	</xacro:if>
-	<xacro:if value="$(arg fd_scanner_enabled)">
-		<xacro:fd_scanner prefix="fd_scanner"
-			robot_namespace="$(arg robot_namespace)"
-			angled="$(arg fd_scanner_angled)"
-			simulated_velodyne="true" />
-		<joint name="fd_scanner_joint" type="fixed">
-			<origin xyz="$(arg fd_scanner_xyz)"
-				rpy="$(arg fd_scanner_rpy)" />
+	<xacro:if value="$(arg velodyne_enabled)">
+		<link name="velodyne_mount">
+			<visual>
+				<geometry>
+					<box size="0.1 0.1 0.1" />
+				</geometry>
+				<material name="black000" />
+			</visual>
+			<collision>
+				<geometry>
+					<box size="0.1 0.1 0.1" />
+				</geometry>
+			</collision>
+			<inertial>
+				<mass value="0.3" />
+				<inertia ixx="1e-3" ixy="1e-3" ixz="1e-3" iyy="1e-3"
+					iyz="1e-3" izz="1e-3" />
+			</inertial>
+		</link>
+		<joint name="velodyne_mount_joint" type="fixed">
+			<origin xyz="0 0 0.05" rpy="0 0 0" />
 			<parent link="top_plate_link" />
-			<child link="fd_scanner_link" />
+			<child link="velodyne_mount" />
 		</joint>
+		<xacro:VLP-16 parent="velodyne_mount" name="velodyne"
+			topic="velodyne_points" hz="10" samples="1875" gpu="true">
+			<origin xyz="0 0 0.05" rpy="0 0 0" />
+		</xacro:VLP-16>
 	</xacro:if>
 	<gazebo>
@@ -248,14 +263,15 @@
 	</gazebo>
 	<gazebo>
-	    <plugin name="p3d_base_controller" filename="libgazebo_ros_p3d.so">
-	      <alwaysOn>true</alwaysOn>
-	      <updateRate>50.0</updateRate>
-	      <bodyName>base_footprint</bodyName>
-	      <topicName>ground_truth/state</topicName>
-	      <gaussianNoise>0.01</gaussianNoise>
-	      <frameName>world</frameName>
-	      <xyzOffsets>0 0 0</xyzOffsets>
-	      <rpyOffsets>0 0 0</rpyOffsets>
-    	</plugin>
+		<plugin name="p3d_base_controller"
+			filename="libgazebo_ros_p3d.so">
+			<alwaysOn>true</alwaysOn>
+			<updateRate>50.0</updateRate>
+			<bodyName>base_footprint</bodyName>
+			<topicName>ground_truth/state</topicName>
+			<gaussianNoise>0.01</gaussianNoise>
+			<frameName>world</frameName>
+			<xyzOffsets>0 0 0</xyzOffsets>
+			<rpyOffsets>0 0 0</rpyOffsets>
+		</plugin>
 	</gazebo>
 </robot>

Commit message: Added launch with ideal robot

File: rrg_nbv_exploration_plugins/urdf/husky.urdf.xacro (robot description, xacro)
@@ -24,32 +24,20 @@
 <robot name="husky" xmlns:xacro="http://ros.org/wiki/xacro">
 	<xacro:arg name="laser_enabled" default="false" />
-	<xacro:arg name="laser_xyz"
-		default="$(optenv HUSKY_LMS1XX_XYZ 0.2206 0.0 0.00635)" />
-	<xacro:arg name="laser_rpy"
-		default="$(optenv HUSKY_LMS1XX_RPY 0.0 0.0 0.0)" />
+	<xacro:arg name="laser_xyz" default="$(optenv HUSKY_LMS1XX_XYZ 0.2206 0.0 0.00635)" />
+	<xacro:arg name="laser_rpy" default="$(optenv HUSKY_LMS1XX_RPY 0.0 0.0 0.0)" />
 	<xacro:arg name="realsense_enabled" default="false" />
-	<xacro:arg name="realsense_xyz"
-		default="$(optenv HUSKY_REALSENSE_XYZ 0 0 0)" />
-	<xacro:arg name="realsense_rpy"
-		default="$(optenv HUSKY_REALSENSE_RPY 0 0 3.14)" />
-	<xacro:property name="husky_front_bumper_extend"
-		value="$(optenv HUSKY_FRONT_BUMPER_EXTEND 0)" />
-	<xacro:property name="husky_rear_bumper_extend"
-		value="$(optenv HUSKY_REAR_BUMPER_EXTEND 0)" />
+	<xacro:arg name="realsense_xyz" default="$(optenv HUSKY_REALSENSE_XYZ 0 0 0)" />
+	<xacro:arg name="realsense_rpy" default="$(optenv HUSKY_REALSENSE_RPY 0 0 3.14)" />
+	<xacro:property name="husky_front_bumper_extend" value="$(optenv HUSKY_FRONT_BUMPER_EXTEND 0)" />
+	<xacro:property name="husky_rear_bumper_extend" value="$(optenv HUSKY_REAR_BUMPER_EXTEND 0)" />
 	<xacro:arg name="velodyne_enabled" default="false" />
 	<xacro:arg name="robot_namespace" default="/" />
 	<!-- Included URDF/XACRO Files -->
-	<xacro:include
-		filename="$(find husky_description)/urdf/decorations.urdf.xacro" />
-	<xacro:include
-		filename="$(find husky_description)/urdf/wheel.urdf.xacro" />
-	<xacro:include
-		filename="$(find rrg_nbv_exploration_plugins)/urdf/intel_realsense.urdf.xacro" />
-	<xacro:include
-		filename="$(find husky_description)/urdf/accessories/sick_lms1xx_mount.urdf.xacro" />
-	<xacro:include
-		filename="$(find rrg_nbv_exploration_plugins)/urdf/sensor_arch.urdf.xacro" />
-	<xacro:include
-		filename="$(find velodyne_description)/urdf/VLP-16.urdf.xacro" />
+	<xacro:include filename="$(find husky_description)/urdf/decorations.urdf.xacro" />
+	<xacro:include filename="$(find husky_description)/urdf/wheel.urdf.xacro" />
+	<xacro:include filename="$(find rrg_nbv_exploration_plugins)/urdf/intel_realsense.urdf.xacro" />
+	<xacro:include filename="$(find husky_description)/urdf/accessories/sick_lms1xx_mount.urdf.xacro" />
+	<xacro:include filename="$(find rrg_nbv_exploration_plugins)/urdf/sensor_arch.urdf.xacro" />
+	<xacro:include filename="$(find velodyne_description)/urdf/VLP-16.urdf.xacro" />
 	<xacro:property name="M_PI" value="3.14159" />
 	<material name="black000">
@@ -63,6 +51,5 @@
 	<xacro:property name="wheelbase" value="0.5120" />
 	<xacro:property name="track" value="0.5708" />
-	<xacro:property name="wheel_vertical_offset"
-		value="0.03282" />
+	<xacro:property name="wheel_vertical_offset" value="0.03282" />
 	<!-- Wheel Properties -->
 	<xacro:property name="wheel_length" value="0.1143" />
@@ -73,15 +60,11 @@
 			<origin xyz="0 0 0" rpy="0 0 0" />
 			<geometry>
-				<mesh
-					filename="package://husky_description/meshes/base_link.dae" />
+				<mesh filename="package://husky_description/meshes/base_link.dae" />
 			</geometry>
 		</visual>
 		<collision>
-			<origin
-				xyz="${( husky_front_bumper_extend - husky_rear_bumper_extend ) / 2.0} 0 ${base_z_size/4}"
-				rpy="0 0 0" />
+			<origin xyz="${( husky_front_bumper_extend - husky_rear_bumper_extend ) / 2.0} 0 ${base_z_size/4}" rpy="0 0 0" />
 			<geometry>
-				<box
-					size="${ base_x_size + husky_front_bumper_extend + husky_rear_bumper_extend } ${base_y_size} ${base_z_size/2}" />
+				<box size="${ base_x_size + husky_front_bumper_extend + husky_rear_bumper_extend } ${base_y_size} ${base_z_size/2}" />
 			</geometry>
 		</collision>
@@ -89,6 +72,5 @@
 			<origin xyz="0 0 ${base_z_size*3/4-0.01}" rpy="0 0 0" />
 			<geometry>
-				<box
-					size="${base_x_size*4/5} ${base_y_size} ${base_z_size/2-0.02}" />
+				<box size="${base_x_size*4/5} ${base_y_size} ${base_z_size/2-0.02}" />
 			</geometry>
 		</collision>
@@ -97,6 +79,5 @@
 	<link name="base_footprint" />
 	<joint name="base_footprint_joint" type="fixed">
-		<origin xyz="0 0 ${-wheel_vertical_offset + wheel_radius}"
-			rpy="0 0 0" />
+		<origin xyz="0 0 ${-wheel_vertical_offset + wheel_radius}" rpy="0 0 0" />
 		<parent link="base_footprint" />
 		<child link="base_link" />
@@ -107,6 +88,5 @@
 			<mass value="46.034" />
 			<origin xyz="-0.00065 -0.085 0.062" />
-			<inertia ixx="0.6022" ixy="-0.02364" ixz="-0.1197"
-				iyy="1.7386" iyz="-0.001544" izz="2.0296" />
+			<inertia ixx="0.6022" ixy="-0.02364" ixz="-0.1197" iyy="1.7386" iyz="-0.001544" izz="2.0296" />
 		</inertial>
 	</link>
@@ -120,34 +100,26 @@
 	<link name="imu_link" />
 	<joint name="imu_joint" type="fixed">
-		<origin xyz="$(optenv HUSKY_IMU_XYZ 0.19 0 0.149)"
-			rpy="$(optenv HUSKY_IMU_RPY 0 -1.5708 3.1416)" />
+		<origin xyz="$(optenv HUSKY_IMU_XYZ 0.19 0 0.149)" rpy="$(optenv HUSKY_IMU_RPY 0 -1.5708 3.1416)" />
 		<parent link="base_link" />
 		<child link="imu_link" />
 	</joint>
-	<gazebo reference="imu_link">
-	</gazebo>
+	<gazebo reference="imu_link"></gazebo>
 	<!-- Husky wheel macros -->
 	<xacro:husky_wheel wheel_prefix="front_left">
-		<origin
-			xyz="${wheelbase/2} ${track/2} ${wheel_vertical_offset}" rpy="0 0 0" />
+		<origin xyz="${wheelbase/2} ${track/2} ${wheel_vertical_offset}" rpy="0 0 0" />
 	</xacro:husky_wheel>
 	<xacro:husky_wheel wheel_prefix="front_right">
-		<origin
-			xyz="${wheelbase/2} ${-track/2} ${wheel_vertical_offset}" rpy="0 0 0" />
+		<origin xyz="${wheelbase/2} ${-track/2} ${wheel_vertical_offset}" rpy="0 0 0" />
 	</xacro:husky_wheel>
 	<xacro:husky_wheel wheel_prefix="rear_left">
-		<origin
-			xyz="${-wheelbase/2} ${track/2} ${wheel_vertical_offset}" rpy="0 0 0" />
+		<origin xyz="${-wheelbase/2} ${track/2} ${wheel_vertical_offset}" rpy="0 0 0" />
 	</xacro:husky_wheel>
 	<xacro:husky_wheel wheel_prefix="rear_right">
-		<origin
-			xyz="${-wheelbase/2} ${-track/2} ${wheel_vertical_offset}"
-			rpy="0 0 0" />
+		<origin xyz="${-wheelbase/2} ${-track/2} ${wheel_vertical_offset}" rpy="0 0 0" />
 	</xacro:husky_wheel>
 	<xacro:husky_decorate />
 	<xacro:if value="$(arg laser_enabled)">
 		<xacro:sick_lms1xx_mount prefix="base" />
-		<xacro:sick_lms1xx frame="base_laser" topic="scan"
-			robot_namespace="$(arg robot_namespace)" />
+		<xacro:sick_lms1xx frame="base_laser" topic="scan" robot_namespace="$(arg robot_namespace)" />
 		<joint name="laser_mount_joint" type="fixed">
 			<origin xyz="$(arg laser_xyz)" rpy="$(arg laser_rpy)" />
@@ -173,6 +145,5 @@
 			<inertial>
 				<mass value="0.01" />
-				<inertia ixx="1e-3" ixy="1e-3" ixz="1e-3" iyy="1e-3"
-					iyz="1e-3" izz="1e-3" />
+				<inertia ixx="1e-3" ixy="1e-3" ixz="1e-3" iyy="1e-3" iyz="1e-3" izz="1e-3" />
 			</inertial>
 		</link>
@@ -193,6 +164,5 @@
 			</joint>
 		</transmission>
-		<xacro:intel_realsense_mount
-			prefix="camera" topic="camera" parent_link="realsense_mountpoint" />
+		<xacro:intel_realsense_mount prefix="camera" topic="camera" parent_link="realsense_mountpoint" />
 	</xacro:if>
 	<xacro:if value="$(arg velodyne_enabled)">
@@ -211,6 +181,5 @@
 			<inertial>
 				<mass value="0.3" />
-				<inertia ixx="1e-3" ixy="1e-3" ixz="1e-3" iyy="1e-3"
-					iyz="1e-3" izz="1e-3" />
+				<inertia ixx="1e-3" ixy="1e-3" ixz="1e-3" iyy="1e-3" iyz="1e-3" izz="1e-3" />
 			</inertial>
 		</link>
@@ -220,18 +189,15 @@
 			<child link="velodyne_mount" />
 		</joint>
-		<xacro:VLP-16 parent="velodyne_mount" name="velodyne"
-			topic="velodyne_points" hz="10" samples="1875" gpu="true">
+		<xacro:VLP-16 parent="velodyne_mount" name="velodyne" topic="velodyne_points" hz="10" samples="1875" gpu="true">
 			<origin xyz="0 0 0.05" rpy="0 0 0" />
 		</xacro:VLP-16>
 	</xacro:if>
 	<gazebo>
-		<plugin name="gazebo_ros_control"
-			filename="libgazebo_ros_control.so">
+		<plugin name="gazebo_ros_control" filename="libgazebo_ros_control.so">
 			<robotNamespace>$(arg robot_namespace)</robotNamespace>
 		</plugin>
 	</gazebo>
 	<gazebo>
-		<plugin name="imu_controller"
-			filename="libhector_gazebo_ros_imu.so">
+		<plugin name="imu_controller" filename="libhector_gazebo_ros_imu.so">
 			<robotNamespace>$(arg robot_namespace)</robotNamespace>
 			<updateRate>50.0</updateRate>
@@ -247,6 +213,5 @@
 	</gazebo>
 	<gazebo>
-		<plugin name="gps_controller"
-			filename="libhector_gazebo_ros_gps.so">
+		<plugin name="gps_controller" filename="libhector_gazebo_ros_gps.so">
 			<robotNamespace>$(arg robot_namespace)</robotNamespace>
 			<updateRate>40</updateRate>
@@ -263,6 +228,5 @@
 	</gazebo>
 	<gazebo>
-		<plugin name="p3d_base_controller"
-			filename="libgazebo_ros_p3d.so">
+		<plugin name="p3d_base_controller" filename="libgazebo_ros_p3d.so">
 			<alwaysOn>true</alwaysOn>
 			<updateRate>50.0</updateRate>
